File: CalcVox_H2_Schematics.kicad_sch (KiCad schematic)
At the start: 69 parts, among them J1 Battery_Barrel_Jack, J2 AudioJack3_SwitchTR, SW1-25 SW_Push, SW1-26 SW_Push, SW1-27 SW_Push, SW1-28 SW_Push, SW1-29 SW_Push, SW1-30 SW_Push, SW1-31 SW_Push, SW1-32 SW_Push, SW2-25 SW_Push, SW2-26 SW_Push, SW2-27 SW_Push, SW2-28 SW_Push, SW2-29 SW_Push, SW2-30 SW_Push, SW2-31 SW_Push, SW2-32 SW_Push, SW3-25 SW_Push, SW3-26 SW_Push, SW3-27 SW_Push, SW3-28 SW_Push, SW3-29 SW_Push, SW3-30 SW_Push, SW3-31 SW_Push, SW3-32 SW_Push, SW4-25 SW_Push, SW4-26 SW_Push, SW4-27 SW_Push, SW4-28 SW_Push, SW4-29 SW_Push, SW4-30 SW_Push, SW4-31 SW_Push, SW4-32 SW_Push, SW5-25 SW_Push, SW5-26 SW_Push, SW5-27 SW_Push, SW5-28 SW_Push, SW5-29 SW_Push, SW5-30 SW_Push, SW5-31 SW_Push, SW5-32 SW_Push, SW6-25 SW_Push, SW6-26 SW_Push, SW6-27 SW_Push, SW6-28 SW_Push, SW6-29 SW_Push, SW6-30 SW_Push, SW6-31 SW_Push, SW6-32 SW_Push, U1 Teensy4.1, U2 MOUDLE-SEEEDUINO-XIAO-ESP32S3

Commit message: added readme
Parts:
- added AGND-GND1: SolderJumper_2_Open, Jumper:SolderJumper-2_P1.3mm_Open_TrianglePad1.0x1.5mm, symbol Jumper:SolderJumper_2_Open
Connections:
- net GND: now also AGND-GND1.2 (B)
- net at A1.8 (AGND), J2.S, LSLeft1.1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: now also AGND-GND1.1 (A)
Changed lines of the file:
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@@
   (junction (at 184.15 97.79) (diameter 0) (color 0 0 0 0)
   )
+  (junction (at 278.13 215.9) (diameter 0) (color 0 0 0 0)
+  )
   (junction (at 167.64 46.99) (diameter 0) (color 0 0 0 0)
   )
@@
     (stroke (width 0) (type default))
   )
+  (wire (pts (xy 278.13 215.9) (xy 278.13 194.31))
+    (stroke (width 0) (type default))
+  )
   (wire (pts (xy 85.09 95.25) (xy 85.09 97.79))
     (stroke (width 0) (type default))
@@
     (stroke (width 0) (type default))
   )
-  (wire (pts (xy 278.13 226.06) (xy 278.13 194.31))
+  (wire (pts (xy 278.13 226.06) (xy 278.13 215.9))
     (stroke (width 0) (type default))
   )
@@
     (property "Intersheetrefs" "${INTERSHEET_REFS}" (at 112.7058 173.99 0)
       (effects (font (size 1.27 1.27)) (justify right) hide)
+    )
+  )
+  (global_label "GND" (shape input) (at 285.75 215.9 0) (fields_autoplaced)
+    (effects (font (size 1.27 1.27)) (justify left))
+    (property "Intersheetrefs" "${INTERSHEET_REFS}" (at 292.6057 215.9 0)
+      (effects (font (size 1.27 1.27)) (justify left) hide)
     )
   )
@@
     )
   )
+  (symbol (lib_id "Jumper:SolderJumper_2_Open") (at 281.94 215.9 0) (unit 1)
+    (in_bom yes) (on_board yes) (dnp no) (fields_autoplaced)
+    (property "Reference" "AGND-GND1" (at 281.94 209.55 0)
+      (effects (font (size 1.27 1.27)))
+    )
+    (property "Value" "SolderJumper_2_Open" (at 281.94 212.09 0)
+      (effects (font (size 1.27 1.27)))
+    )
+    (property "Footprint" "Jumper:SolderJumper-2_P1.3mm_Open_TrianglePad1.0x1.5mm" (at 281.94 215.9 0)
+      (effects (font (size 1.27 1.27)) hide)
+    )
+    (property "Datasheet" "~" (at 281.94 215.9 0)
+      (effects (font (size 1.27 1.27)) hide)
+    )
+    (pin "1")
+    (pin "2")
+    (instances
+      (project "CalcVox_H2_Schematics"
+        (path "/b7dd3139-7adc-48fa-8dea-095b900fd75c"
+          (reference "AGND-GND1") (unit 1)
+        )
+      )
+    )
+  )
   (symbol (lib_id "Device:Speaker") (at 284.48 238.76 0) (unit 1)
     (in_bom yes) (on_board yes) (dnp no) (fields_autoplaced)
@@
     )
     (property "Footprint" "Connector_Audio:Jack_3.5mm_CUI_SJ1-3524N_Horizontal" (at 248.92 209.55 0)
-      (effects (font (size 1.27 1.27)))
+      (effects (font (size 1.27 1.27)) hide)
     )
     (property "Datasheet" "~" (at 248.92 209.55 0)
@@
     )
     (property "Footprint" "XIAO:MOUDLE14P-SMD-2.54-21X17.8MM" (at 255.27 163.83 0)
-      (effects (font (size 1.27 1.27)) (justify bottom))
+      (effects (font (size 1.27 1.27)) (justify bottom) hide)
     )
     (property "Datasheet" "" (at 255.27 163.83 0)

Commit message: Added 3d models and fixed small mistakes
Parts:
- SW1-25, SW1-26, SW1-27, SW1-28, SW1-29, SW1-30, SW1-31, SW1-32, SW2-25, SW2-26, SW2-27, SW2-28, SW2-29, SW2-30, SW2-31, SW2-32, SW3-25, SW3-26, SW3-27, SW3-28, SW3-29, SW3-30, SW3-31, SW3-32, SW4-25, SW4-26, SW4-27, SW4-28, SW4-29, SW4-30, SW4-31, SW4-32, SW5-25, SW5-26, SW5-27, SW5-28, SW5-29, SW5-30, SW5-31, SW5-32, SW6-25, SW6-26, SW6-27, SW6-28, SW6-29, SW6-30, SW6-31, SW6-32, SWReset1: footprint Button_Switch_THT:SW_PUSH_6mm_H7.3mm_1 -> Button_Switch_THT:SW_PUSH_6mm_H9.5mm

Commit message: updated with feedback
Parts:
- added C1: 10µF, Capacitor_THT:C_Disc_D6.0mm_W2.5mm_P5.00mm, symbol Device:C
- added C2, C3, C4: 0.1µF, Capacitor_THT:C_Disc_D6.0mm_W2.5mm_P5.00mm, symbol Device:C
Connections:
- net 5V: now also C1.2
- net ESP_3V3: now also C4.1
- net GND: now also C1.1, C2.2, C3.2, C4.2
- net at D1.1 (K), U1.48 (VIN): now also C2.1
- net at D2.1 (K), U2.14 (5V): now also C3.1
Other:
- moved on the sheet: D1, D2
